File: game-boy-zero-link-board.kicad_sch (KiCad schematic)
At the start: 6 parts, among them J1 GBA_Link, J2 DMG_Link, J3 Breakout, SW1 SW_SPDT, U1 Pico_Reduced, U2 BOB-12009

Commit message: commit local changes (untested)
Parts:
- removed SW1: SW_SPDT, Connector_PinHeader_2.54mm:PinHeader_1x03_P2.54mm_Vertical, symbol Switch:SW_SPDT
- removed U1: Pico_Reduced, MCU_RaspberryPi_and_Boards:RPi_Pico_SMD_TH_REDUCED, symbol MCU_RaspberryPi_and_Boards:Pico_Reduced
- added U1: RP2040-Zero, MCU_RaspberryPi_and_Boards:RP2040-Zero_SMD_TH, symbol MCU_RaspberryPi_and_Boards:RP2040-Zero
- J3: value Breakout -> GB_IDC_port; footprint Connector_PinHeader_2.54mm:PinHeader_1x06_P2.54mm_Vertical -> gb-link-socket:GameBoy_LinkPort_DMG_MGB_IDC_Horizontal; symbol Connector:Conn_01x06_Pin -> Connector:Conn_01x07_Pin
Connections:
- net GND1 is gone; now on net GND: J1.6 (Pin_6), J2.6 (Pin_6), J3.6 (Pin_6), U2.10 (GND_2)
- net VCCLOGIC is gone; now on net GBVCC: U2.9 (HV)
- net +3.3V: now also U1.21 (3V3)
- net GND: now also J3.SH, U1.22 (GND)
- net PSC: now also U1.1 (GPIO0)
- net PSD: now also U1.4 (GPIO3)
- net PSI: now also U1.2 (GPIO1)
- net PSO: now also U1.3 (GPIO2)
- no-connect marks 26 -> 0
Other:
- note removed: "MODE SWITCH"
